Commit message: first (front) sonar has been imported, and works fine

File: mymobibot_description/urdf/macros.xacro (robot description, xacro)
@@ -48,5 +48,5 @@
           <parent link="chassis"/>
           <child link="${lr}_wheel"/>
-          <origin xyz="${+wheelPos-chassisLength/4} ${tY*wheelWidth/2+tY*chassisWidth/2} ${wheelRadius}" rpy="0 0 0" />
+          <origin xyz="${-wheelPos+chassisLength/4} ${tY*wheelWidth/2+tY*chassisWidth/2} ${wheelRadius}" rpy="0 0 0" />
           <axis xyz="0 1 0" rpy="0 0 0" />
           <limit effort="100" velocity="100"/>

File: mymobibot_description/urdf/mymobibot.xacro (robot description, xacro)
@@ -12,6 +12,10 @@
   <xacro:property name="wheelPos" value="0.2"/>
   <xacro:property name="wheelMass" value="5"/>
-  <xacro:property name="cameraSize" value="0.05"/>
-  <xacro:property name="cameraMass" value="0.1"/>
+  <!--xacro:property name="cameraSize" value="0.05"/>
+  <xacro:property name="cameraMass" value="0.1"/-->
+  <xacro:property name="sonarHeight" value="0.025"/>
+  <xacro:property name="sonarLength" value="0.005"/>
+  <xacro:property name="sonarWidth" value="0.05"/>
+  <xacro:property name="sonarMass" value="0.1"/>
   <xacro:include filename="$(find mymobibot_description)/urdf/mymobibot.gazebo" />
   <xacro:include filename="$(find mymobibot_description)/urdf/materials.xacro" />
@@ -48,5 +52,5 @@
   <link name="caster_wheel">
     <collision>
-      <origin xyz="${casterRadius-chassisLength/2} 0 ${casterRadius-chassisHeight+wheelRadius}" rpy="0 0 0"/>
+      <origin xyz="${-casterRadius+chassisLength/2} 0 ${casterRadius-chassisHeight+wheelRadius}" rpy="0 0 0"/>
       <geometry>
 	<sphere radius="${casterRadius}"/>
@@ -54,5 +58,5 @@
     </collision>
     <visual>
-      <origin xyz="${casterRadius-chassisLength/2} 0 ${casterRadius-chassisHeight+wheelRadius}" rpy="0 0 0"/>
+      <origin xyz="${-casterRadius+chassisLength/2} 0 ${casterRadius-chassisHeight+wheelRadius}" rpy="0 0 0"/>
       <geometry>
 	<sphere radius="${casterRadius}"/>
@@ -60,5 +64,5 @@
     </visual>
     <inertial>
-      <origin xyz="${casterRadius-chassisLength/2} 0 ${casterRadius-chassisHeight+wheelRadius}" rpy="0 0 0"/>
+      <origin xyz="${-casterRadius+chassisLength/2} 0 ${casterRadius-chassisHeight+wheelRadius}" rpy="0 0 0"/>
       <mass value="${casterMass}"/>
       <xacro:sphere_inertia m="${casterMass}" r="${casterRadius}"/>
@@ -67,5 +71,5 @@
   <xacro:wheel lr="left" tY="-1"/>
   <xacro:wheel lr="right" tY="1"/>
-  <joint name="camera_joint" type="fixed">
+  <!--joint name="camera_joint" type="fixed">
     <origin xyz="${-cameraSize+chassisLength/2} 0 ${cameraSize+wheelRadius+cameraSize/2}" rpy="0 0 0"/>
     <parent link="chassis"/>
@@ -91,4 +95,30 @@
       <xacro:box_inertia m="${cameraMass}" x="${cameraSize}" y="${cameraSize}" z="${cameraSize}" />
     </inertial>
+  </link-->
+  <joint name="sonar_front_joint" type="fixed">
+    <!--axis xyz="0 1 0" /-->
+    <origin xyz="${chassisLength/2-sonarLength/2} 0 ${wheelRadius/2+chassisHeight+sonarHeight/2}" rpy="0 0 0"/>
+    <parent link="chassis"/>
+    <child link="base_sonar_front"/>
+  </joint>
+  <link name="base_sonar_front">
+    <collision>
+      <origin xyz="0 0 0" rpy="0 0 0"/>
+      <geometry>
+        <box size="${sonarLength} ${sonarWidth} ${sonarHeight}"/>
+      </geometry>
+    </collision>
+    <visual>
+      <origin xyz="0 0 0" rpy="0 0 0"/>
+      <geometry>
+        <box size="${sonarLength} ${sonarWidth} ${sonarHeight}"/>
+      </geometry>
+      <material name="blue"/>
+    </visual>
+    <inertial>
+      <mass value="${sonarMass}" />
+      <origin xyz="0 0 0" rpy="0 0 0"/>
+      <xacro:box_inertia m="${sonarMass}" x="${sonarLength}" y="${sonarWidth}" z="${sonarHeight}" />
+    </inertial>
   </link>
 </robot>
